Commit message: Sync env/base/utils chain with lab repo (feat/el_4090_2)
- base: legged_robot(+rew_mixin, multi-stage reward curriculum), base_task,
  legged_robot_config synced from lab
- spider_nomal: EL_4090 env/configs synced; port fork's DELAY control branch
  in _compute_torques; symmetry.py/ReadMe.md synced
- elspider_air: elspider.py/elspider_raycast.py/configs synced from lab;
  add lab's elspider_tasks.py (Pose/FootTrack/LoadAdapt/Stand subclasses)
- pd_gru_lidar task imported verbatim from lab; enable multi_stage_rewards
  on El4090LidarCfg (spider cfg carries stage-list scales with the flag off,
  which crashes _prepare_reward_function - latent bug in lab too)
- utils: terrain.py from lab + legacy curved/trapezoid/_draw_circle kept at
  tail (direct-call only) + getattr fallback for stepping_stones fields
  (configs shadowing LeggedRobotCfg.terrain); math_utils/helpers/logger synced;
  LidarSensor moved in-package (warp-only build from lab)
- scripts/play.py from lab (keyboard input, follow camera); keep fork's
  train.py (cfg snapshot dump) and play_laptop.py
- resources: el_4090.urdf from lab (meshes already identical)
- batch_rollout rew_mixin / franka_batch_rollout synced

File: legged_gym/resources/robots/el_4090/urdf/el_4090.urdf (robot description, URDF)
Before this commit: robot el_4090, 25 links, 24 joints
Joints:
- joint LB_HAA: limit lower=-1.57 upper=1.57 effort=80 velocity=15.8 -> lower=-3 upper=3 effort=80 velocity=15.8
- joint LB_HFE: limit lower=-1.57 upper=1.57 effort=80 velocity=15.8 -> lower=-3 upper=3 effort=80 velocity=15.8
- joint LB_KFE: limit lower=-1.57 upper=1.57 effort=80 velocity=15.8 -> lower=-3 upper=3 effort=80 velocity=15.8
- joint LF_HAA: limit lower=-1.57 upper=1.57 effort=80 velocity=15.8 -> lower=-3 upper=3 effort=80 velocity=15.8
- joint LF_HFE: limit lower=-1.57 upper=1.57 effort=80 velocity=15.8 -> lower=-3 upper=3 effort=80 velocity=15.8
- joint LF_KFE: limit lower=-1.57 upper=1.57 effort=80 velocity=15.8 -> lower=-3 upper=3 effort=80 velocity=15.8
- joint LM_HAA: limit lower=-1.57 upper=1.57 effort=80 velocity=15.8 -> lower=-3 upper=3 effort=80 velocity=15.8
- joint LM_HFE: limit lower=-1.57 upper=1.57 effort=80 velocity=15.8 -> lower=-3 upper=3 effort=80 velocity=15.8
- joint LM_KFE: limit lower=-1.57 upper=1.57 effort=80 velocity=15.8 -> lower=-3 upper=3 effort=80 velocity=15.8
- joint RB_HAA: limit lower=-1.57 upper=1.57 effort=80 velocity=15.8 -> lower=-3 upper=3 effort=80 velocity=15.8
- joint RB_HFE: limit lower=-1.57 upper=1.57 effort=80 velocity=15.8 -> lower=-3 upper=3 effort=80 velocity=15.8
- joint RB_KFE: limit lower=-1.57 upper=1.57 effort=80 velocity=15.8 -> lower=-3 upper=3 effort=80 velocity=15.8
- joint RF_HAA: limit lower=-1.57 upper=1.57 effort=80 velocity=15.8 -> lower=-3 upper=3 effort=80 velocity=15.8
- joint RF_HFE: limit lower=-1.57 upper=1.57 effort=80 velocity=15.8 -> lower=-3 upper=3 effort=80 velocity=15.8
- joint RF_KFE: limit lower=-1.57 upper=1.57 effort=80 velocity=15.8 -> lower=-3 upper=3 effort=80 velocity=15.8
- joint RM_HAA: limit lower=-1.57 upper=1.57 effort=80 velocity=15.8 -> lower=-3 upper=3 effort=80 velocity=15.8
- joint RM_HFE: limit lower=-1.57 upper=1.57 effort=80 velocity=15.8 -> lower=-3 upper=3 effort=80 velocity=15.8
- joint RM_KFE: limit lower=-1.57 upper=1.57 effort=80 velocity=15.8 -> lower=-3 upper=3 effort=80 velocity=15.8
